File: STK-681-332-E EvalBoard OwnRoutingStarted.brd (EAGLE design)
At the start: 160 x 100 mm, 39 parts, among them P1 10K, Q1 BS250, T1 SR5A0, T2 SR5A0, T3 BC546B, T4 BC546B, T5 BC546B, T6 BC546B, U1 STK681_332E, X1 MKDS3/2-5.08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

Commit message: Add files via upload
Parts:
- moved C1 156.3 mm to (41.9, 74.9)
- moved C2 156.3 mm to (36.8, 59.7)
- moved C3 156.3 mm to (30.5, 59.7)
- moved C4 156.3 mm to (41.9, 59.7)
- moved C5 156.3 mm to (35.6, 74.9)
- moved C6 156.3 mm to (48.3, 74.9)
- moved D1 156.3 mm to (17.8, 62.2)
- moved J1 156.3 mm to (128.3, 47.0)
- moved J2 156.3 mm to (147.3, 64.8)
- moved J3 156.3 mm to (137.2, 76.2)
- moved LED1 156.3 mm to (30.5, 71.1)
- moved LED2 156.3 mm to (21.6, 58.4)
- moved LED3 156.3 mm to (50.8, 54.6)
- moved P1 156.3 mm to (115.6, 66.0)
- moved Q1 156.3 mm to (50.8, 59.7)
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